Commit message: Made changes to how meshes are refernced in the urdf

File: install/quori_description/share/quori_description/urdf/quori.xacro (robot description, xacro)
@@ -1,91 +1 @@
-<?xml version="1.0"?>
-<robot name="quori" xmlns:xacro="http://www.ros.org/wiki/xacro">
-  <xacro:include filename="$(find quori_description)/urdf/quori_kinematics.xacro" />
-  <xacro:include filename="$(find quori_description/urdf/ramsis_kinematics.xacro" />
-  <quori_kinematics />
-  <ramsis_kinematics />
-  <material name="blue">
-    <color rgba="0 0 0.8 1"/>
-  </material>
-  <material name="black">
-    <color rgba="0 0 0 1"/>
-  </material>
-  <material name="white">
-    <color rgba="1 1 1 1"/>
-  </material>
-  <material name="gray">
-    <color rgba="0.5 0.5 0.5 1"/>
-  </material>
-  <!-- Join the quori robot to the ramsis robot's turret joint -->
-  <joint name="ramsis_quori_connector" type="fixed">
-    <parent link="ramsis/turret_link" />
-    <child link="quori/base_link"/>
-  </joint>
-  <link name="world"/>
-  <joint name="fixed" type="fixed">
-    <parent link="world"/>
-    <child link="ramsis/wheel_axle"/>
-  </joint>
-  <xacro:macro name="joint_transmission" params="prefix">
-    <transmission name="${prefix}_tran">
-      <type>transmission_interface/SimpleTransmission</type>
-      <actuator name="${prefix}_motor">
-        <hardwareInterface>hardware_interface/PositionJointInterface</hardwareInterface>
-        <mechanicalReduction>1</mechanicalReduction>
-      </actuator>
-      <joint name="${prefix}">
-        <hardwareInterface>hardware_interface/PositionJointInterface</hardwareInterface>
-      </joint>
-    </transmission>
-  </xacro:macro>
-  <xacro:macro name="wheel_transmission" params="prefix">
-    <transmission name="${prefix}_tran">
-      <type>transmission_interface/SimpleTransmission</type>
-      <actuator name="${prefix}_motor">
-        <hardwareInterface>hardware_interface/VelocityJointInterface</hardwareInterface>
-        <mechanicalReduction>1</mechanicalReduction>
-      </actuator>
-      <joint name="${prefix}">
-        <hardwareInterface>hardware_interface/VelocityJointInterface</hardwareInterface>
-      </joint>
-    </transmission>
-  </xacro:macro>
-  <xacro:joint_transmission prefix="waist_pitch"/>
-  <xacro:joint_transmission prefix="r_shoulder_pitch"/>
-  <xacro:joint_transmission prefix="r_shoulder_roll"/>
-  <xacro:joint_transmission prefix="l_shoulder_pitch"/>
-  <xacro:joint_transmission prefix="l_shoulder_roll"/>
-  <xacro:wheel_transmission prefix="l_wheel"/>
-  <xacro:wheel_transmission prefix="r_wheel"/>
-  <xacro:joint_transmission prefix="turret"/>
-  <gazebo reference="quori/body_upper">
-    <material>Gazebo/White</material>
-  </gazebo>
-  <gazebo reference="quori/base_link">
-    <material>Gazebo/White</material>
-  </gazebo>
-  <gazebo reference="quori/head">
-    <material>Gazebo/White</material>
-  </gazebo>
-  <gazebo reference="quori/r_arm_upper">
-    <material>Gazebo/White</material>
-  </gazebo>
-  <gazebo reference="quori/r_arm_lower">
-    <material>Gazebo/White</material>
-  </gazebo>
-  <gazebo reference="quori/l_arm_upper">
-    <material>Gazebo/White</material>
-  </gazebo>
-  <gazebo reference="quori/l_arm_lower">
-    <material>Gazebo/White</material>
-  </gazebo>
-  <gazebo reference="base_link_diff">
-    <material>Gazebo/White</material>
-  </gazebo>
-  <gazebo>
-    <plugin name="gazebo_ros_control" filename="libgazebo_ros_control.so">
-      <!-- <robotNamespace>/quori</robotNamespace> -->
-      <robotSimType>gazebo_ros_control/DefaultRobotHWSim</robotSimType>
-    </plugin>
-  </gazebo>
-</robot>
+/home/jorge/quori_ws/src/quori_description/urdf/quori.xacro

File: install/quori_description/share/quori_description/urdf/quori_kinematics.xacro (robot description, xacro)
@@ -1,261 +1 @@
-<?xml version="1.0"?>
-<xacro:macro name="quori_kinematics" xmlns:xacro="http://ros.org/wiki/xacro">
-  <link name="quori/base_link">
-    <inertial>
-      <origin xyz="0 0 0.23" rpy="0 0 0"/>
-      <mass value="2"/>
-      <inertia ixx="0.052"  ixy="0"  ixz="0" iyy="0.052" iyz="0" izz="0.031" />
-    </inertial>
-    <visual>
-      <origin rpy="0 0 -1.57079632679" xyz="0.02 0 -0.2007174"/>
-      <geometry>
-        <mesh filename="file:///home/jorge/quori_ws/src/quori_description/meshes/180915_Lower_Torso.dae"/>
-      </geometry>
-    </visual>
-  </link>
-  <link name="quori/body_upper">
-    <inertial>
-      <origin xyz="0 0 -0.01" rpy="0 0 0"/>
-      <mass value="26.75"/>
-      <inertia ixx="2.5"  ixy="0"  ixz="0" iyy="2.5" iyz="0" izz="0.134" />
-    </inertial>
-    <visual>
-      <origin rpy="0 0 -1.57079632679" xyz="0.02 0 -0.5476974"/>
-      <geometry>
-        <mesh filename="file:///home/jorge/quori_ws/src/quori_description/meshes/10917_Upper_Torso+Waist.dae"/>
-      </geometry>
-    </visual>
-  </link>
-  <joint name="waist_pitch" type="revolute">
-    <origin xyz="0 0 0.34798" rpy="0 0 0"/>
-    <parent link="quori/base_link"/>
-    <child link="quori/body_upper"/>
-    <axis xyz="0 -1 0" />
-    <limit lower="-0.47123889803846897" upper="0.2111848394913139" effort="1" velocity="1"/>
-  </joint>
-  <link name="quori/r_shoulder">
-    <inertial>
-      <origin xyz="0 0 0" rpy="0 0 0"/>
-      <mass value="0.01"/>
-      <inertia ixx="0.01"  ixy="0"  ixz="0" iyy="0.0" iyz="0" izz="0.0" />
-    </inertial>
-  </link>
-  <joint name="r_shoulder_pitch" type="revolute">
-    <origin xyz="0.015 -0.16403066 0.43021758" rpy="0 0 0"/>
-    <parent link="quori/body_upper"/>
-    <child link="quori/r_shoulder"/>
-    <axis xyz="0 -1 0" />
-    <limit lower="-2.4" upper="2.4" effort="1" velocity="1"/>
-  </joint>
-  <link name="quori/r_arm_upper">
-    <inertial>
-      <origin xyz="0 0 0" rpy="0 0 0"/>
-      <mass value="0.01"/>
-      <inertia ixx="0.1"  ixy="0"  ixz="0" iyy="0.0" iyz="0" izz="0.0" />
-    </inertial>
-    <visual>
-      <origin rpy="-1.57079632679 0 0" xyz="0.165 -0.9765 -0.137"/>
-      <geometry>
-        <mesh filename="file:///home/jorge/quori_ws/src/quori_description/meshes/10917_Upper_Arm+gear_right.dae"/>
-      </geometry>
-    </visual>
-  </link>
-  <joint name="r_shoulder_roll" type="revolute">
-    <origin xyz="0 0 0" rpy="0 0 0" />
-    <parent link="quori/r_shoulder" />
-    <child link="quori/r_arm_upper" />
-    <axis xyz="-1 0 0" />
-    <limit lower="-1.1" upper="1.1" effort="1" velocity="1" />
-  </joint>
-  <link name="quori/r_arm_upper2lower">
-    <inertial>
-      <origin xyz="0 0 0.3" rpy="0 0 0"/>
-      <mass value="0.19"/>
-      <inertia ixx="0.006"  ixy="0"  ixz="0" iyy="0.006" iyz="0" izz="0.0" />
-    </inertial>
-    <visual>
-    <origin rpy="-1.57079632679 0 0" xyz="0 -0.13 0"/>
-      <geometry>
-        <cylinder length="0.08" radius="0.015"/>
-      </geometry>
-      <material name="white"/>
-    </visual>
-  </link>
-  <joint name="r_arm_upper2lower_j" type="fixed">
-    <parent link="quori/r_arm_upper"/>
-    <child link="quori/r_arm_upper2lower"/>
-  </joint>
-  <link name="quori/r_arm_lower">
-    <inertial>
-      <origin xyz="0 0 0" rpy="0 0 0"/>
-      <mass value="0.01"/>
-      <inertia ixx="0.1"  ixy="0"  ixz="0" iyy="0.0" iyz="0" izz="0.0" />
-    </inertial>
-    <visual>
-      <origin rpy="1.570759635 1.570759635 0" xyz="0 0 0"/>
-      <geometry>
-        <mesh filename="file:///home/jorge/quori_ws/src/quori_description/meshes/10917_Lower_Arm_right.dae" />
-      </geometry>
-    </visual>
-  </link>
-  <joint name="r_elbow_pitch" type="fixed">
-    <origin xyz="0 -0.15 0" rpy="0 0 0" />
-    <parent link="quori/r_arm_upper" />
-    <child link="quori/r_arm_lower" />
-  </joint>
-  <link name="quori/l_shoulder">
-    <inertial>
-      <origin xyz="0 0 0" rpy="0 0 0"/>
-      <mass value="0.1"/>
-      <inertia ixx="0.1"  ixy="0"  ixz="0" iyy="0.0" iyz="0" izz="0.0" />
-    </inertial>
-  </link>
-  <joint name="l_shoulder_pitch" type="revolute">
-    <origin xyz="0.015 0.16403066 0.43021758" rpy="0 0 0" />
-    <parent link="quori/body_upper" />
-    <child link="quori/l_shoulder" />
-    <axis xyz="0 -1 0" />
-    <limit lower="-2.4" upper="2.4" effort="1" velocity="1" />
-  </joint>
-  <link name="quori/l_arm_upper">
-    <inertial>
-      <origin xyz="0 0 0" rpy="0 0 0" />
-      <mass value="0.01" />
-      <inertia ixx="0.1"  ixy="0"  ixz="0" iyy="0.0" iyz="0" izz="0.0" />
-    </inertial>
-    <visual>
-      <origin rpy="-1.57079632679 0 -3.14" xyz="0.165 0.9765 -0.137" />
-      <geometry>
-        <mesh filename="file:///home/jorge/quori_ws/src/quori_description/meshes/10917_Upper_Arm+gear_left.dae"/>
-      </geometry>
-    </visual>
-  </link>
-  <joint name="l_shoulder_roll" type="revolute">
-    <origin xyz="0 0 0" rpy="0 0 0" />
-    <parent link="quori/l_shoulder" />
-    <child link="quori/l_arm_upper" />
-    <axis xyz="1 0 0" />
-    <limit lower="-1.1" upper="1.1" effort="1" velocity="1" />
-  </joint>
-  <link name="quori/l_arm_upper2lower">
-    <inertial>
-      <origin xyz="0 0 0.3" rpy="0 0 0"/>
-      <mass value="0.19"/>
-      <inertia ixx="0.006"  ixy="0"  ixz="0" iyy="0.006" iyz="0" izz="0.0" />
-    </inertial>
-    <visual>
-    <origin rpy="-1.57079632679 0 0" xyz="0 0.13 0"/>
-      <geometry>
-        <cylinder length="0.08" radius="0.015"/>
-      </geometry>
-      <material name="white"/>
-    </visual>
-  </link>
-  <joint name="l_arm_upper2lower_j" type="fixed">
-    <parent link="quori/l_arm_upper"/>
-    <child link="quori/l_arm_upper2lower"/>
-  </joint>
-  <link name="quori/l_arm_lower">
-    <inertial>
-      <origin xyz="0 0 0" rpy="0 0 0"/>
-      <mass value="0.01"/>
-      <inertia ixx="0.1"  ixy="0"  ixz="0" iyy="0.0" iyz="0" izz="0.0" />
-    </inertial>
-    <visual>
-      <origin rpy="-1.570759635 -1.570759635 0" xyz="0 0 0" />
-      <geometry>
-        <mesh filename="file:///home/jorge/quori_ws/src/quori_description/meshes/10917_Lower_Arm_left.dae" />
-      </geometry>
-    </visual>
-  </link>
-  <joint name="l_elbow_pitch" type="fixed">
-    <origin xyz="0 0.15 0" rpy="0 0 0"/>
-    <parent link="quori/l_arm_upper"/>
-    <child link="quori/l_arm_lower"/>
-  </joint>
-  <link name="quori/head">
-    <inertial>
-      <origin xyz="0 0 0" rpy="0 0 0"/>
-      <mass value="1.9"/>
-      <inertia ixx="0.008"  ixy="0"  ixz="0" iyy="0.0056" iyz="0" izz="0.0056" />
-    </inertial>
-    <visual>
-      <origin rpy="0 0 -1.57079632679" xyz="0.01 0 -1.11" />
-      <geometry>
-        <mesh filename="file:///home/jorge/quori_ws/src/quori_description/meshes/10917_Helmet_Duripod.dae" />
-      </geometry>
-    </visual>
-  </link>
-  <link name="quori/face">
-    <visual>
-      <origin xyz="0 0 0.085" />
-      <geometry>
-        <sphere radius="0.1" />
-      </geometry>
-      <material name="white" />
-    </visual>
-  </link>
-  <joint name="head_swivel" type="fixed">
-    <parent link="quori/head" />
-    <child link="quori/face" />
-  </joint>
-  <gazebo reference="quori/face">
-    <visual>
-      <plugin name="faceplugin" filename="libfaceplugin.so">
-      <robotNamespace>quori</robotNamespace>
-        <height>120</height>
-        <width>240</width>
-      </plugin>
-    </visual>
-  </gazebo>
-  <joint name="neck" type="fixed">
-    <origin xyz="0 0 0.554" rpy="0 0 0" />
-    <parent link="quori/body_upper" />
-    <child link="quori/head" />
-  </joint>
-  <joint name="head_camera_optical_joint" type="fixed">
-    <origin xyz="0 0 0" rpy="-1.57079632679 0 -1.57079632679" />
-    <parent link="quori/head_camera" />
-    <child link="quori/head_camera_optical" />
-  </joint>
-  <link name="quori/head_camera_optical">
-  </link>
-  <link name="quori/head_camera">
-    <inertial>
-      <origin xyz="0 0 0" rpy="0 0 0"/>
-      <mass value="0.3"/>
-      <inertia ixx="0.0004"  ixy="0"  ixz="0" iyy="0.0001" iyz="0" izz="0.0004" />
-    </inertial>
-    <visual>
-      <geometry>
-        <box size="0.04 0.11 0.04"/>
-      </geometry>
-      <origin rpy="0 0 0" xyz="0 0 -0"/>
-      <material name="black"/>
-    </visual>
-  </link>
-  <joint name="camera_pitch" type="fixed">
-    <origin xyz="0.055 0 0.21" rpy="0 0 0" />
-    <parent link="quori/head" />
-    <child link="quori/head_camera" />
-  </joint>
-  <link name="quori/head_mic">
-    <inertial>
-      <origin xyz="0 0 0" rpy="0 0 0"/>
-      <mass value="0.05"/>
-      <inertia ixx="0.1"  ixy="0"  ixz="0" iyy="0.0" iyz="0" izz="0.0" />
-    </inertial>
-    <visual>
-      <geometry>
-        <cylinder length="0.002" radius="0.03"/>
-      </geometry>
-      <origin rpy="0 0 0" xyz="0 0 -0"/>
-      <material name="blue"/>
-    </visual>
-  </link>
-  <joint name="mic_array" type="fixed">
-    <origin xyz="-0.008 0 0.218" rpy="0 -.3 0" />
-    <parent link="quori/head" />
-    <child link="quori/head_mic" />
-  </joint>
-</xacro:macro>
+/home/jorge/quori_ws/src/quori_description/urdf/quori_kinematics.xacro

File: install/quori_description/share/quori_description/urdf/quori_standalone.xacro (robot description, xacro)
@@ -1,5 +1 @@
-<?xml version="1.0"?>
-<robot name="quori" xmlns:xacro="http://www.ros.org/wiki/xacro">
-  <xacro:include filename="$(find quori_description)/urdf/quori_kinematics.xacro" />
-  <quori_kinematics />
-</robot>
+/home/jorge/quori_ws/src/quori_description/urdf/quori_standalone.xacro

File: install/quori_description/share/quori_description/urdf/ramsis_kinematics.xacro (robot description, xacro)
@@ -1,107 +1 @@
-<?xml version="1.0"?>
-<xacro:macro name="ramsis_kinematics" xmlns:xacro="http://ros.org/wiki/xacro">
-  <material name="ramsis/base_link_material">
-    <color rgba="0 0 0 1"/>
-  </material>
-  <material name="ramsis/laser_scanner_material">
-    <color rgba="0.3 0.3 0.3 1"/>
-  </material>
-  <link name="ramsis/base_link_diff">
-    <inertial>
-      <origin xyz="0 0 0.1013587" rpy="0 0 0"/>
-      <mass value="9.8"/>
-      <inertia ixx="0.176"  ixy="0"  ixz="0" iyy="0.176" iyz="0" izz="0.285" />
-    </inertial>
-    <visual>
-      <origin xyz="0 0 0.1013587" rpy="0 0 0" />
-      <geometry>
-        <cylinder length="0.2027174" radius="0.2413"/>
-      </geometry>
-      <material name="ramsis/base_link_material"/>
-    </visual>
-  </link>
-  <link name="ramsis/base_laser_scanner">
-    <inertial>
-      <mass value="0.17"/>
-      <inertia ixx="0.0001"  ixy="0"  ixz="0" iyy="0.0001" iyz="0" izz="0.0001" />
-    </inertial>
-    <visual>
-        <geometry>
-          <cylinder length="0.025" radius="0.05"/>
-      </geometry>
-      <origin rpy="0 0 0" xyz="0 0 -0"/>
-      <material name="ramsis/laser_scanner_material"/>
-    </visual>
-  </link>
-  <joint name="laser_scanner_joint" type="fixed">
-    <origin xyz="0.152 0 0.156" rpy="0 0.0 -1.5707" />
-    <parent link="ramsis/base_link_diff" />
-    <child link="ramsis/base_laser_scanner" />
-  </joint>
-  <link name="ramsis/turret_link">
-    <inertial>
-      <origin xyz="0 0 0" rpy="0 0 0"/>
-      <mass value="0.01"/>
-      <inertia ixx="0.01"  ixy="0"  ixz="0" iyy="0.0" iyz="0" izz="0.0" />
-    </inertial>
-  </link>
-  <link name="ramsis/base_link">
-    <inertial>
-      <origin xyz="0 0 0" rpy="0 0 0"/>
-      <mass value="0.01"/>
-      <inertia ixx="0.01"  ixy="0"  ixz="0" iyy="0.0" iyz="0" izz="0.0" />
-    </inertial>
-  </link>
-  <link name="ramsis/l_wheel_link">
-    <inertial>
-      <origin xyz="0 0 0" rpy="0 0 0"/>
-      <mass value="0.1"/>
-      <inertia ixx="0.1"  ixy="0"  ixz="0" iyy="0.0" iyz="0" izz="0.0" />
-    </inertial>
-  </link>
-  <link name="ramsis/r_wheel_link">
-    <inertial>
-      <origin xyz="0 0 0" rpy="0 0 0"/>
-      <mass value="0.1"/>
-      <inertia ixx="0.1"  ixy="0"  ixz="0" iyy="0.0" iyz="0" izz="0.0" />
-    </inertial>
-  </link>
-  <joint name="ramsis/wheel_axle_joint" type="fixed">
-    <origin xyz="0.1 0 -0.075" />
-    <parent link="ramsis/wheel_axle" />
-    <child link="ramsis/base_link_diff" />
-  </joint>
-  <joint name="turret2base" type="fixed">
-    <origin xyz="0 0 -0.2027174" />
-    <parent link="ramsis/turret_link" />
-    <child link="ramsis/base_link" />
-  </joint>
-  <link name="ramsis/wheel_axle">
-    <inertial>
-      <origin xyz="0 0 0" rpy="0 0 0"/>
-      <mass value="0.00"/>
-      <inertia ixx="0.00"  ixy="0"  ixz="0" iyy="0.0" iyz="0" izz="0.0" />
-    </inertial>
-  </link>
-  <joint name="l_wheel" type="continuous">
-    <origin xyz="0 0.12284075 0" rpy="0 0 0"/>
-    <parent link="ramsis/wheel_axle"/>
-    <child link="ramsis/l_wheel_link"/>
-    <axis xyz="0 1 0" />
-    <limit effort="1" velocity="0.5"/>
-  </joint>
-  <joint name="r_wheel" type="continuous">
-    <origin xyz="0 -0.12284075 0" rpy="0 0 0"/>
-    <parent link="ramsis/wheel_axle"/>
-    <child link="ramsis/r_wheel_link"/>
-    <axis xyz="0 1 0" />
-    <limit effort="1" velocity="0.5"/>
-  </joint>
-  <joint name="turret" type="continuous">
-    <origin xyz="0 0 0.2027174" rpy="0 0 0"/>
-    <parent link="ramsis/base_link_diff"/>
-    <child link="ramsis/turret_link"/>
-    <axis xyz="0 0 1" />
-    <limit effort="1" velocity="3"/>
-  </joint>
-</xacro:macro>
+/home/jorge/quori_ws/src/quori_description/urdf/ramsis_kinematics.xacro

File: install/quori_description/share/quori_description/urdf/ramsis_standalone.xacro (robot description, xacro)
@@ -1,5 +1 @@
-<?xml version="1.0"?>
-<robot name="ramsis" xmlns:xacro="http://www.ros.org/wiki/xacro">
-  <xacro:include filename="$(find quori_description)/urdf/ramsis_kinematics.xacro" />
-  <ramsis_kinematics />
-</robot>
+/home/jorge/quori_ws/src/quori_description/urdf/ramsis_standalone.xacro

File: src/quori_description/urdf/quori.urdf (robot description, URDF)
Before this commit: robot quori, 23 links, 22 joints
Links:
- link quori/base_link: geometry visual mesh filename=model://quori/meshes/180915_Lower_Torso.dae
- link quori/body_upper: geometry visual mesh filename=model://quori/meshes/0917_Upper_Torso+Waist.dae
- link quori/head: geometry visual mesh filename=model://quori/meshes/0917_Helmet_Duripod.dae
- link quori/l_arm_lower: geometry visual mesh filename=model://quori/meshes/0917_Lower_Arm_left.dae
- link quori/l_arm_upper: geometry visual mesh filename=model://quori/meshes/0917_Upper_Arm+gear_left.dae
- link quori/r_arm_lower: geometry visual mesh filename=model://quori/meshes/0917_Lower_Arm_right.dae
- link quori/r_arm_upper: geometry visual mesh filename=model://quori/meshes/0917_Upper_Arm+gear_right.dae

File: src/quori_description/urdf/quori_kinematics.xacro (robot description, xacro)
@@ -10,5 +10,5 @@
       <origin rpy="0 0 -1.57079632679" xyz="0.02 0 -0.2007174"/>
       <geometry>
-        <mesh filename="file:///home/jorge/quori_ws/src/quori_description/meshes/180915_Lower_Torso.dae"/>
+        <mesh filename="model://quori/meshes/180915_Lower_Torso.dae"/>
       </geometry>
     </visual>
@@ -23,5 +23,5 @@
       <origin rpy="0 0 -1.57079632679" xyz="0.02 0 -0.5476974"/>
       <geometry>
-        <mesh filename="file:///home/jorge/quori_ws/src/quori_description/meshes/10917_Upper_Torso+Waist.dae"/>
+        <mesh filename="model://quori/meshes/10917_Upper_Torso+Waist.dae"/>
       </geometry>
     </visual>
@@ -57,5 +57,5 @@
       <origin rpy="-1.57079632679 0 0" xyz="0.165 -0.9765 -0.137"/>
       <geometry>
-        <mesh filename="file:///home/jorge/quori_ws/src/quori_description/meshes/10917_Upper_Arm+gear_right.dae"/>
+        <mesh filename="model://quori/meshes/10917_Upper_Arm+gear_right.dae"/>
       </geometry>
     </visual>
@@ -95,5 +95,5 @@
       <origin rpy="1.570759635 1.570759635 0" xyz="0 0 0"/>
       <geometry>
-        <mesh filename="file:///home/jorge/quori_ws/src/quori_description/meshes/10917_Lower_Arm_right.dae" />
+        <mesh filename="model://quori/meshes/10917_Lower_Arm_right.dae" />
       </geometry>
     </visual>
@@ -127,5 +127,5 @@
       <origin rpy="-1.57079632679 0 -3.14" xyz="0.165 0.9765 -0.137" />
       <geometry>
-        <mesh filename="file:///home/jorge/quori_ws/src/quori_description/meshes/10917_Upper_Arm+gear_left.dae"/>
+        <mesh filename="model://quori/meshes/10917_Upper_Arm+gear_left.dae"/>
       </geometry>
     </visual>
@@ -165,5 +165,5 @@
       <origin rpy="-1.570759635 -1.570759635 0" xyz="0 0 0" />
       <geometry>
-        <mesh filename="file:///home/jorge/quori_ws/src/quori_description/meshes/10917_Lower_Arm_left.dae" />
+        <mesh filename="model://quori/meshes/10917_Lower_Arm_left.dae" />
       </geometry>
     </visual>
@@ -183,5 +183,5 @@
       <origin rpy="0 0 -1.57079632679" xyz="0.01 0 -1.11" />
       <geometry>
-        <mesh filename="file:///home/jorge/quori_ws/src/quori_description/meshes/10917_Helmet_Duripod.dae" />
+        <mesh filename="model://quori/meshes/10917_Helmet_Duripod.dae" />
       </geometry>
     </visual>
